File: stm8l151k6t6_board.kicad_sch (KiCad schematic)
At the start: 31 parts, among them J1 Conn_01x08, J2 Conn_01x08, J3 Conn_01x08, J4 Conn_01x08, J5 Conn_01x04, SW1 RESET, SW2 USER, U1 USB_B_Micro, U2 TPMIC5504, U3 STM8L151K6T6, Y1 8MHz, Y2 32K768Hz

Commit message: updated version
Parts:
- removed J1, J2, J3, J4: Conn_01x08, Connector_PinHeader_2.54mm:PinHeader_1x08_P2.54mm_Vertical, symbol Connector_Generic:Conn_01x08
- added C1, C3, C6: 100nF, Capacitor_SMD:C_0402_1005Metric, symbol Device:C_Small
- added J1, J3: Conn_01x16, Connector_PinHeader_2.54mm:PinHeader_1x16_P2.54mm_Vertical, symbol Connector_Generic:Conn_01x16
- added R2, R3: 27, Resistor_SMD:R_0805_2012Metric, symbol Device:R
- added U3: FT230XQ, Package_DFN_QFN:QFN-16-1EP_4x4mm_P0.65mm_EP2.1x2.1mm, symbol Interface_USB:FT230XQ
- H1, H2, H3, H4: footprint MountingHole:MountingHole_3.2mm_M3 -> MountingHole:MountingHole_2.2mm_M2
- R1: value 100 -> 1k; LCSC C5139650 -> (none)
- R4: renamed from R2; value 100 -> 1k; LCSC C5139650 -> (none)
- R5: renamed from R3; value 100 -> 1K
- renumbered C7 to C10, C9 to C11, C8 to C12, C10 to C13, C1 to C2, C2 to C4, C3 to C5, C4 to C7, C5 to C8, C6 to C9, J5 to J2, U3 to U4
Connections:
- net +3V3: now also C3.1, C6.1, J1.3 (Pin_3), U3.1 (VCCIO), U3.9 (~{RESET})
- net +5V: now also C1.1, J1.1 (Pin_1), U3.10 (VCC)
- net GND: now also C1.2, C3.2, C6.2, J1.2 (Pin_2), J1.4 (Pin_4), U3.13 (GND), U3.17 (GND), U3.3 (GND)
- net PA4: now also J1.14 (Pin_14)
- net PA5: now also J1.15 (Pin_15)
- net PA6: now also J1.16 (Pin_16)
- net PB0: now also J3.12 (Pin_12)
- net PB1: now also J3.11 (Pin_11)
- net PB2: now also J3.10 (Pin_10)
- net PB3: now also J3.9 (Pin_9)
- net PB4: now also J3.8 (Pin_8)
- net PB5: now also J3.7 (Pin_7)
- net PB6: now also J3.6 (Pin_6)
- net PB7: now also J3.5 (Pin_5)
- net PC0: now also J1.5 (Pin_5)
- net PC1: now also J1.6 (Pin_6)
- net PC4: now also J1.9 (Pin_9)
- net PD0: now also J3.16 (Pin_16)
- net PD1: now also J3.15 (Pin_15)
- net PD2: now also J3.14 (Pin_14)
- net PD3: now also J3.13 (Pin_13)
- net PD4: now also J3.4 (Pin_4)
- net PD5: now also J3.3 (Pin_3)
- net PD6: now also J3.2 (Pin_2)
- net PD7: now also J3.1 (Pin_1)
- net USB_D+: now reaches U1.2 (D-)
- net USB_D+: now also R3.1
- net USB_D-: now reaches U1.3 (D+)
- net USB_D-: now also R2.1
- net PA0 renamed PA0/SWIM
- net PA0/SWIM: now also J1.10 (Pin_10)
- net PA1 renamed PA1/RST
- net PA1/RST: now also J1.11 (Pin_11)
- net PC2 renamed USART_RX
- net USART_RX: now also J1.7 (Pin_7), U3.15 (TXD)
- net PC3 renamed USART_TX
- net USART_TX: now also J1.8 (Pin_8), U3.2 (RXD)
- new net: R3.2, U3.6 (USBDP)
- new net: R2.2, U3.7 (USBDM)
- no-connect marks 5 -> 10
Other:
- company: (none) -> Andres Bravo
- title: (none) -> STM8L151 Dev Board
- moved on the sheet: J2, U1, U4
